Commit message: resnet

File: 16811/urdf/m6.urdf (robot description, URDF)
Before this commit: robot m6, 37 links, 36 joints
Links:
- removed link color
- removed link depth
- removed link ired1
- removed link ired2
- removed link rs200_camera
- link base1__INPUT_INTERFACE: geometry collision box size=0.106400 0.069500 0.031050; visual mesh filename=/home/yihe/Spring2020/16811/meshes/M6_base_motor.STL
- link base2__INPUT_INTERFACE: geometry collision box size=0.106400 0.069500 0.031050; visual mesh filename=/home/yihe/Spring2020/16811/meshes/M6_base_motor.STL
- link base3__INPUT_INTERFACE: geometry collision box size=0.106400 0.069500 0.031050; visual mesh filename=/home/yihe/Spring2020/16811/meshes/M6_base_motor.STL
- link base4__INPUT_INTERFACE: geometry collision box size=0.106400 0.069500 0.031050; visual mesh filename=/home/yihe/Spring2020/16811/meshes/M6_base_motor.STL
- link base5__INPUT_INTERFACE: geometry collision box size=0.106400 0.069500 0.031050; visual mesh filename=/home/yihe/Spring2020/16811/meshes/M6_base_motor.STL
- link base6__INPUT_INTERFACE: geometry collision box size=0.106400 0.069500 0.031050; visual mesh filename=/home/yihe/Spring2020/16811/meshes/M6_base_motor.STL
- link base_link: geometry collision box size=0.073 0.075 0.046; collision box size=0.073 0.075 0.046
- link camera_mount: geometry visual mesh filename=/home/yihe/Spring2020/16811/meshes/camera_mount.STL
- link elbow1__INPUT_INTERFACE: geometry collision box size=0.05950 0.04800 0.037500; collision box size=0.06850 0.06500 0.037500
- link elbow2__INPUT_INTERFACE: geometry collision box size=0.05950 0.04800 0.037500; collision box size=0.06850 0.06500 0.037500
- link elbow3__INPUT_INTERFACE: geometry collision box size=0.05950 0.04800 0.037500; collision box size=0.06850 0.06500 0.037500
- link elbow4__INPUT_INTERFACE: geometry collision box size=0.05950 0.04800 0.037500; collision box size=0.06850 0.06500 0.037500
- link elbow5__INPUT_INTERFACE: geometry collision box size=0.05950 0.04800 0.037500; collision box size=0.06850 0.06500 0.037500
- link elbow6__INPUT_INTERFACE: geometry collision box size=0.05950 0.04800 0.037500; collision box size=0.06850 0.06500 0.037500
- link leg1__LAST_LINK: geometry collision box size=0.045000 0.047030 0.047030; collision box size=0.05850 0.04800 0.03650
- link leg2__LAST_LINK: geometry collision box size=0.045000 0.047030 0.047030; collision box size=0.05850 0.04800 0.03650
- link leg3__LAST_LINK: geometry collision box size=0.045000 0.047030 0.047030; collision box size=0.05850 0.04800 0.03650
- link leg4__LAST_LINK: geometry collision box size=0.045000 0.047030 0.047030; collision box size=0.05850 0.04800 0.03650
- link leg5__LAST_LINK: geometry collision box size=0.045000 0.047030 0.047030; collision box size=0.05850 0.04800 0.03650
- link leg6__LAST_LINK: geometry collision box size=0.045000 0.047030 0.047030; collision box size=0.05850 0.04800 0.03650
- link shoulder1__INPUT_INTERFACE: geometry collision box size=0.108140 0.04500 0.104000; visual mesh filename=/home/yihe/Spring2020/16811/meshes/M6_left_link1_red.STL
- link shoulder2__INPUT_INTERFACE: geometry collision box size=0.108140 0.04500 0.104000; visual mesh filename=/home/yihe/Spring2020/16811/meshes/M6_right_link1_red.STL
- link shoulder3__INPUT_INTERFACE: geometry collision box size=0.108140 0.04500 0.104000; visual mesh filename=/home/yihe/Spring2020/16811/meshes/M6_left_link1_red.STL
- link shoulder4__INPUT_INTERFACE: geometry collision box size=0.108140 0.04500 0.104000; visual mesh filename=/home/yihe/Spring2020/16811/meshes/M6_right_link1_red.STL
- link shoulder5__INPUT_INTERFACE: geometry collision box size=0.108140 0.04500 0.104000; visual mesh filename=/home/yihe/Spring2020/16811/meshes/M6_left_link1_red.STL
- link shoulder6__INPUT_INTERFACE: geometry collision box size=0.108140 0.04500 0.104000; visual mesh filename=/home/yihe/Spring2020/16811/meshes/M6_right_link1_red.STL
Joints:
- removed joint color_joint
- removed joint depth_joint
- removed joint ired1_joint
- removed joint ired2_joint
- removed joint realsense_joint
